Commit message: add imu to urdf & switch to cpu laser

File: src/rosbot_description/urdf/rosbot.xacro (robot description, xacro)
@@ -339,3 +339,10 @@
   </joint>
   <link name="range_rr"></link>
+  <joint name="imu_joint" type="fixed">
+    <axis xyz="0 1 0" />
+    <origin xyz="-0.1 0 0" rpy="0 0 0"/>
+    <parent link="top"/>
+    <child link="imu_link"/>
+  </joint>
+  <link name="imu_link"></link>
 </robot>

Commit message: remove imu in urdf (just realised real robot is using the same xacro file)

File: src/rosbot_description/urdf/rosbot.xacro (robot description, xacro)
@@ -339,10 +339,3 @@
   </joint>
   <link name="range_rr"></link>
-  <joint name="imu_joint" type="fixed">
-    <axis xyz="0 1 0" />
-    <origin xyz="-0.1 0 0" rpy="0 0 0"/>
-    <parent link="top"/>
-    <child link="imu_link"/>
-  </joint>
-  <link name="imu_link"></link>
 </robot>
